File: hardware/pcb/hedwig.brd (EAGLE design)
At the start: 60 x 60 mm, 85 parts, among them J1 DX07B024JJ1R1500, P1 JTAG-10MINI, P2 SENSOR_SCL, P3 RF_SCK, P4 PC1, P5 PC5, P6 PC9, Q1 16MHz, Q2 IRLML6402, Q3 20V/0.2A/8MHz/1.2Ω/1Vth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

Commit message: latest board - square, logo
Routing:
- net N$27: track 11.9 -> 12.6 mm
- net GND: track 30.7 -> 29.9 mm, vias 38 -> 67
