File: hardware/pcb/hedwig/hedwig.sch (EAGLE design)
At the start: 85 parts, among them J1 DX07B024JJ1R1500, P1 JTAG-10MINI, P2 SENSOR_SCL, P3 RF_SCK, P4 PC1, P5 PC5, P6 PC9, Q1 16MHz, Q2 IRLML6402, Q3 20V/0.2A/8MHz/1.2Ω/1Vth, Q6 20V/0.2A/8MHz/1.2Ω/1Vth, U1 NRF24L01SMD, U2 TEXAS_INSTRUMENTS_TLC59731DRT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, U3 FT232RQ, U4 TPS7A26-1.8, U5 ADP2302, U6 9DoF IMU, U7 MPL3115A2LGA, X1 8M, X2 32.768

Commit message: Added pics, pdf, fixed silkscreen, and added more vias
Other:
- note added: "1.8V Power Supply"
- note added: "3.3V Power Supply"
- note removed: "3.3V to 1.8V Conversion"
- note removed: "5V to 3.3V Conversion"
Changed lines of the file:
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@@
 <plain>
 <text x="-161.798" y="107.442" size="5.08" layer="91">Outputs and Input Selection</text>
-<text x="-55.88" y="106.68" size="5.08" layer="91">5V to 3.3V Conversion</text>
-<text x="-160.02" y="22.86" size="5.08" layer="91">3.3V to 1.8V Conversion</text>
+<text x="-53.34" y="106.68" size="5.08" layer="91">3.3V Power Supply</text>
+<text x="-160.02" y="20.32" size="5.08" layer="91">1.8V Power Supply</text>
 </plain>
 <instances>

Commit message: Fix major issues in hardware
Parts:
- C10, C11, C8, C9: value 0.1uF -> 8.2pF
- C14: value 0.1uF -> 2.2uF
Connections:
- removed net N$25: 5V_BAT.P, Q2.D
- new net N$34: 5V_BAT.P, Q2.S
- net +3V3: now also U$1.VDDA/VREF+
- net +5V: no longer Q2.S
- net GND: now also U$1.VSSA/VREF-
- net USB_VCC: now also J1.B_VBUS
Other:
- moved on the sheet: 5V, D3, R10
Changed lines of the file:
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@@
 <part name="X1" library="FaBo-Crystal" deviceset="CRYSTAL" device="-NX3225GD" value="8M"/>
 <part name="GND7" library="supply1" library_urn="urn:adsk.eagle:library:371" deviceset="GND" device=""/>
-<part name="C8" library="SparkFun-Capacitors" deviceset="0.1UF" device="-0603-25V-(+80/-20%)" value="0.1uF"/>
-<part name="C9" library="SparkFun-Capacitors" deviceset="0.1UF" device="-0603-25V-(+80/-20%)" value="0.1uF"/>
+<part name="C8" library="SparkFun-Capacitors" deviceset="0.1UF" device="-0603-25V-(+80/-20%)" value="8.2pF"/>
+<part name="C9" library="SparkFun-Capacitors" deviceset="0.1UF" device="-0603-25V-(+80/-20%)" value="8.2pF"/>
 <part name="X2" library="NDK - NX3215SA-32.768K-STD-MUA-8" deviceset="NX32" device="" value="32.768"/>
-<part name="C10" library="SparkFun-Capacitors" deviceset="0.1UF" device="-0603-25V-(+80/-20%)" value="0.1uF"/>
-<part name="C11" library="SparkFun-Capacitors" deviceset="0.1UF" device="-0603-25V-(+80/-20%)" value="0.1uF"/>
+<part name="C10" library="SparkFun-Capacitors" deviceset="0.1UF" device="-0603-25V-(+80/-20%)" value="8.2pF"/>
+<part name="C11" library="SparkFun-Capacitors" deviceset="0.1UF" device="-0603-25V-(+80/-20%)" value="8.2pF"/>
 <part name="U3" library="FT232RQ" deviceset="FT232RQ" device=""/>
 <part name="J1" library="DX07B024JJ1R1500" deviceset="DX07B024JJ1R1500" device=""/>
@@
 <part name="+3V7" library="supply1" library_urn="urn:adsk.eagle:library:371" deviceset="+3V3" device=""/>
 <part name="GND" library="testpad" library_urn="urn:adsk.eagle:library:385" deviceset="TP" device="B2,54" package3d_urn="urn:adsk.eagle:package:27948/1"/>
-<part name="C14" library="SparkFun-Capacitors" deviceset="0.1UF" device="-0603-25V-(+80/-20%)" value="0.1uF"/>
+<part name="C14" library="SparkFun-Capacitors" deviceset="0.1UF" device="-0603-25V-(+80/-20%)" value="2.2uF"/>
 <part name="D1" library="SFT722N-S" deviceset="SFT722N-S" device=""/>
 <part name="U2" library="Texas Instruments - TLC59731DR" deviceset="TEXAS_INSTRUMENTS_TLC59731DR" device="TEXAS_INSTRUMENTS_TLC59731DR_0_0"/>
@@
 <pinref part="GND32" gate="1" pin="GND"/>
 <wire x1="-53.34" y1="48.26" x2="-53.34" y2="45.72" width="0.1524" layer="91"/>
+<pinref part="U$1" gate="G$1" pin="VSSA/VREF-"/>
+<wire x1="-38.1" y1="40.64" x2="-45.72" y2="40.64" width="0.1524" layer="91"/>
+<wire x1="-45.72" y1="40.64" x2="-45.72" y2="45.72" width="0.1524" layer="91"/>
+<wire x1="-45.72" y1="45.72" x2="-53.34" y2="45.72" width="0.1524" layer="91"/>
+<junction x="-53.34" y="45.72"/>
 </segment>
 </net>
@@
 <junction x="-53.34" y="55.88"/>
 <pinref part="C28" gate="G$1" pin="2"/>
+<pinref part="U$1" gate="G$1" pin="VDDA/VREF+"/>
+<wire x1="-38.1" y1="38.1" x2="-78.74" y2="38.1" width="0.1524" layer="91"/>
+<wire x1="-78.74" y1="38.1" x2="-78.74" y2="55.88" width="0.1524" layer="91"/>
+<wire x1="-78.74" y1="55.88" x2="-63.5" y2="55.88" width="0.1524" layer="91"/>
+<junction x="-63.5" y="55.88"/>
 </segment>
 <segment>
@@
 <label x="15.24" y="50.8" size="1.524" layer="95"/>
 </segment>
+<segment>
+<pinref part="J1" gate="G$1" pin="B_VBUS"/>
+<wire x1="60.96" y1="30.48" x2="66.04" y2="30.48" width="0.1524" layer="91"/>
+<label x="66.04" y="30.48" size="1.778" layer="95"/>
+</segment>
 </net>
 <net name="N$26" class="0">
@@
 <attribute name="VALUE" x="-73.66" y="71.12" size="1.778" layer="96"/>
 </instance>
-<instance part="R10" gate="G$1" x="-83.82" y="55.88" smashed="yes" rot="R90">
-<attribute name="NAME" x="-85.344" y="55.88" size="1.778" layer="95" font="vector" rot="R90" align="bottom-center"/>
-<attribute name="VALUE" x="-82.296" y="55.88" size="1.778" layer="96" font="vector" rot="R90" align="top-center"/>
-</instance>
-<instance part="GND30" gate="1" x="-83.82" y="45.72" smashed="yes">
-<attribute name="VALUE" x="-86.36" y="43.18" size="1.778" layer="96"/>
-</instance>
-<instance part="P+3" gate="1" x="-76.2" y="88.9" smashed="yes">
-<attribute name="VALUE" x="-78.74" y="83.82" size="1.778" layer="96" rot="R90"/>
-</instance>
-<instance part="D3" gate="G$1" x="-93.98" y="81.28" smashed="yes">
-<attribute name="NAME" x="-91.44" y="81.7626" size="1.778" layer="95"/>
-<attribute name="VALUE" x="-91.44" y="78.9686" size="1.778" layer="96"/>
-</instance>
-<instance part="5V" gate="G$1" x="-83.82" y="88.9" smashed="yes">
-<attribute name="NAME" x="-85.09" y="90.17" size="1.778" layer="95"/>
-<attribute name="TP_SIGNAL_NAME" x="-82.55" y="87.63" size="1.778" layer="97"/>
+<instance part="R10" gate="G$1" x="-83.82" y="66.04" smashed="yes" rot="R90">
+<attribute name="NAME" x="-85.344" y="66.04" size="1.778" layer="95" font="vector" rot="R90" align="bottom-center"/>
+<attribute name="VALUE" x="-82.296" y="66.04" size="1.778" layer="96" font="vector" rot="R90" align="top-center"/>
+</instance>
+<instance part="GND30" gate="1" x="-83.82" y="58.42" smashed="yes">
+<attribute name="VALUE" x="-86.36" y="55.88" size="1.778" layer="96"/>
+</instance>
+<instance part="P+3" gate="1" x="-63.5" y="55.88" smashed="yes">
+<attribute name="VALUE" x="-66.04" y="50.8" size="1.778" layer="96" rot="R90"/>
+</instance>
+<instance part="D3" gate="G$1" x="-81.28" y="48.26" smashed="yes">
+<attribute name="NAME" x="-78.74" y="48.7426" size="1.778" layer="95"/>
+<attribute name="VALUE" x="-78.74" y="45.9486" size="1.778" layer="96"/>
+</instance>
+<instance part="5V" gate="G$1" x="-71.12" y="55.88" smashed="yes">
+<attribute name="NAME" x="-72.39" y="57.15" size="1.778" layer="95"/>
+<attribute name="TP_SIGNAL_NAME" x="-69.85" y="54.61" size="1.778" layer="97"/>
 </instance>
 <instance part="FRAME1" gate="G$1" x="-170.18" y="-58.42" smashed="yes">
@@
 <pinref part="R10" gate="G$1" pin="1"/>
 <pinref part="GND30" gate="1" pin="GND"/>
-<wire x1="-83.82" y1="48.26" x2="-83.82" y2="50.8" width="0.1524" layer="91"/>
 </segment>
 <segment>
@@
 <net name="+5V" class="0">
 <segment>
-<pinref part="Q2" gate="G$1" pin="S"/>
-<wire x1="-76.2" y1="76.2" x2="-76.2" y2="81.28" width="0.1524" layer="91"/>
 <pinref part="P+3" gate="1" pin="+5V"/>
 <pinref part="D3" gate="G$1" pin="C"/>
-<wire x1="-76.2" y1="81.28" x2="-76.2" y2="86.36" width="0.1524" layer="91"/>
-<wire x1="-91.44" y1="81.28" x2="-83.82" y2="81.28" width="0.1524" layer="91"/>
-<junction x="-76.2" y="81.28"/>
+<wire x1="-63.5" y1="48.26" x2="-63.5" y2="53.34" width="0.1524" layer="91"/>
+<wire x1="-78.74" y1="48.26" x2="-71.12" y2="48.26" width="0.1524" layer="91"/>
 <pinref part="5V" gate="G$1" pin="TP"/>
-<wire x1="-83.82" y1="81.28" x2="-76.2" y2="81.28" width="0.1524" layer="91"/>
-<wire x1="-83.82" y1="81.28" x2="-83.82" y2="86.36" width="0.1524" layer="91"/>
-<junction x="-83.82" y="81.28"/>
+<wire x1="-71.12" y1="48.26" x2="-63.5" y2="48.26" width="0.1524" layer="91"/>
+<wire x1="-71.12" y1="48.26" x2="-71.12" y2="53.34" width="0.1524" layer="91"/>
+<junction x="-71.12" y="48.26"/>
 </segment>
 <segment>
@@
 <net name="USB_VCC" class="0">
 <segment>
-<pinref part="D3" gate="G$1" pin="A"/>
 <label x="-111.76" y="73.66" size="1.524" layer="95"/>
 <pinref part="Q2" gate="G$1" pin="G"/>
 <pinref part="R10" gate="G$1" pin="2"/>
-<wire x1="-83.82" y1="73.66" x2="-83.82" y2="60.96" width="0.1524" layer="91"/>
+<wire x1="-83.82" y1="73.66" x2="-83.82" y2="71.12" width="0.1524" layer="91"/>
 <wire x1="-111.76" y1="73.66" x2="-96.52" y2="73.66" width="0.1524" layer="91"/>
 <junction x="-83.82" y="73.66"/>
+<pinref part="D3" gate="G$1" pin="A"/>
 <wire x1="-96.52" y1="73.66" x2="-83.82" y2="73.66" width="0.1524" layer="91"/>
-<wire x1="-96.52" y1="81.28" x2="-96.52" y2="73.66" width="0.1524" layer="91"/>
+<wire x1="-83.82" y1="48.26" x2="-96.52" y2="48.26" width="0.1524" layer="91"/>
+<wire x1="-96.52" y1="48.26" x2="-96.52" y2="73.66" width="0.1524" layer="91"/>
 <junction x="-96.52" y="73.66"/>
-</segment>
-</net>
-<net name="N$25" class="0">
-<segment>
-<pinref part="5V_BAT" gate="P" pin="P"/>
-<pinref part="Q2" gate="G$1" pin="D"/>
-<wire x1="-144.78" y1="63.5" x2="-76.2" y2="63.5" width="0.1524" layer="91"/>
-<wire x1="-76.2" y1="63.5" x2="-76.2" y2="66.04" width="0.1524" layer="91"/>
 </segment>
 </net>
@@
 </segment>
 </net>
+<net name="N$34" class="0">
+<segment>
+<pinref part="5V_BAT" gate="P" pin="P"/>
+<wire x1="-144.78" y1="63.5" x2="-116.84" y2="63.5" width="0.1524" layer="91"/>
+<wire x1="-116.84" y1="63.5" x2="-116.84" y2="83.82" width="0.1524" layer="91"/>
+<pinref part="Q2" gate="G$1" pin="S"/>
+<wire x1="-116.84" y1="83.82" x2="-76.2" y2="83.82" width="0.1524" layer="91"/>
+<wire x1="-76.2" y1="83.82" x2="-76.2" y2="76.2" width="0.1524" layer="91"/>
+</segment>
+</net>

Commit message: schematic and pcb update
Parts:
- removed BLTP, GLTP, RLTP: TPB1,27, testpad:TPB1,27
- removed GND_BAT: (no value), wirepad:2,54/1,0
- removed J$1: SMA_EDGE, SparkFun:SMA_EDGE
- removed P2: SENSOR_SCL, falcon:STAG_CONN
- removed P3: RF_SCK, falcon:STAG_CONN
- removed P4: PC1, falcon:STAG_CONN
- removed P5: PC5, falcon:STAG_CONN
- removed P6: PC9, falcon:STAG_CONN
- removed Q1: 16MHz, SparkFun:CRYSTAL5X3
- removed U$2: PUSHBUTTON, falcon:PUSHBUTTON
- added C25: 0.1uF, SparkFun-Capacitors:0.1UF-0603-25V-(+80/-20%)
- added C29: 10nF, SparkFun:CAP0402
- added C30, C34: 0.1uF, SparkFun:CAP0402
- added C31: 1nF, SparkFun:CAP0402
- added C32: 0.3pF, SparkFun:CAP0402
- added C33: 220pF, SparkFun:CAP0402
- added CE, IRQ, MISO, MOSI, SCK, SS: TPB1,27, testpad:TPB1,27
- added D4: DIODE_0603, falcon:DIODE_0603
- added J2: USB4110-GF-A, USB4110-GF-A:USB4110-GF-A
- added J3: SMA_EDGE, SparkFun:SMA_EDGE
- added LED1: (no value), led:LEDCHIPLED_1206
- added R13, R17: 10k, SparkFun-Resistors:2.49KOHM-0603-1/10W-1%
- added R15, R16: 10k, SparkFun:RESISTOR0402
- added R6: 10k, SparkFun-Resistors:10KOHM-0603-1/10W-1%
- added U10: 2450LP14A100T, 2450LP14A100T:2450LP14A100T
- added U9: ICM-20948, ICM-20948:ICM-20948
- added X3: ABM8-16.000MHZ-B2-T, ABM8-16.000MHZ-B2-T:ABM8-16.000MHZ-B2-T
- C10, C11, C8, C9: device SparkFun-Capacitors:0.1UF-0603-25V-(+80/-20%) -> falcon:CAPACITOR_0603
- C12, C13: value 0.1µF -> 0.1uF; device microbuilder:CAP_CERAMIC0805-NOOUTLINE -> falcon:CAPACITOR_0603
- C19: value 0.1uF -> 0.22uF
- C20, C21: value 47uF -> 0.22uF
- C22, C23: value 47uF -> 4.7uF
- D1: value SFT722N-S -> EVERLIGHT_EAST1616RGBB2EVERLIGHT_EAST1616RGBB2_0_0; device SFT722N-S:SFT722N-S -> Everlight - EAST1616RGBB2:EVERLIGHT_EAST1616RGBB2EVERLIGHT_EAST1616RGBB2_0_0
- D3: value SURS8360BT3G -> DIODE_0603; device falcon:DIODE -> falcon:DIODE_0603
- GND: value TPB2,54 -> (none); device testpad:TPB2,54 -> wirepad:2,54/1,0
- J1: value DX07B024JJ1R1500 -> PUSHBUTTON; device DX07B024JJ1R1500:DX07B024JJ1R1500 -> falcon:PUSHBUTTON
- L1: value 3.9nH -> 8.2nH
- L3: value 8.2nH -> 3.9nH
- R10, R12, R14: value 2.49k -> 10k
- R9: value 100k -> 10k
- U6: value 9DoF IMU -> RFX2401C; device SparkFun-Sensors:ICM-20948 -> RFX2401C:RFX2401C
- renumbered 5V_BAT to VBAT, U$1 to U8, U$4 to L4
Connections:
- removed net ADSD_STUB: U6.AD0/SDO
- removed net ANT: C6.2, C7.2, J$1.SIGNAL
- removed net N$7: C4.1, C5.1, L2.1, U1.VDD_PA
- removed net PC6: P5.@2, U8.PC6
- removed net REGOUT: C15.1, U6.REGOUT
- new net 5V_BAT: D4.A, VBAT.P
- new net ALT_IRQ_1: U7.INT1, U8.PA9
- new net ALT_IRQ_2: U7.INT2, U8.PA10
- new net IMU_IRQ: U8.PA8, U9.INT1
- new net N$25: LED1.C, R6.2
- new net N$37: C32.1, U10.IN, U6.ANT
- new net N$39: C15.1, U9.REGOUT
- new net N$53: J3.SIGNAL, U10.OUT
- new net N$57: R16.1, U6.RXEN
- new net N$58: R15.1, U6.TXEN
- new net PC0: U8.PC0
- new net TXRX: C6.2, C7.2, U6.TXRX
- new net VDD_PA: C4.1, C5.1, L2.1, R15.2, U1.VDD_PA
- net +3V3: now also C12.1, C25.2, C29.1, C30.1, C31.1, C33.2, C34.2, D1.COMMON_ANODE, LED1.A, R13.2, R17.2, U6.VDD; no longer C13.1, D1.BA, D1.GA, D1.RA
- net +5V: now also Q2.D
- net 1V8: now also U9.!CS, U9.VDD, U9.VDDIO; no longer U6.!CS, U6.VDD, U6.VDDIO
- net CAP: now also C13.1; no longer C12.1
- net GND: now also C10.2, C11.2, C25.1, C29.2, C30.2, C31.2, C32.2, C33.1, C34.1, C8.2, C9.2, GND.P, J1.OUT@1, J1.OUT@2, J2.GND, J3.GND@0, J3.GND@1, J3.GND@2, J3.GND@3, R6.1, U10.GND, U9.AD0/SDO, U9.FSYNC, U9.GND, U9.RESV_20, X3.GND; no longer C10.1, C11.1, C8.1, C9.1, GND.TP, GND_BAT.P, J$1.GND@0, J$1.GND@1, J$1.GND@2, J$1.GND@3, J1.GNDA, J1.GNDB, J1.SHIELD, U$2.OUT@1, U$2.OUT@2
- net N$1: now also X3.1; no longer Q1.1
- net N$10: now also C8.1; no longer C9.2
- net N$11: now also D1.RED_CATHODE; no longer BLTP.TP, D1.BC
- net N$12: now also D1.BLUE_CATHODE; no longer D1.RC, RLTP.TP
- net N$13: now also C11.1; no longer C10.2
- net N$14: now also C10.1; no longer C11.2
- net N$15: now also J2.CC2; no longer J1.CC2
- net N$2: now also X3.3; no longer Q1.2
- net N$21: now also J2.DP1; no longer J1.DA+
- net N$22: now also J2.DN1; no longer J1.DA-
- net N$26: now also J2.CC1; no longer J1.CC1
- net N$27: now also D1.GREEN_CATHODE; no longer D1.GC, GLTP.TP
- net N$3: now also L1.1; no longer L3.1
- net N$34: now also D4.C; no longer VBAT.P
- net N$6: now also L1.2, L3.1; no longer L1.1, L3.2
- net N$8: now also C9.1; no longer C8.2
- net N$9: now also L3.2; no longer L1.2
- net NRST: now also J1.IN@1, J1.IN@2; no longer U$2.IN@1, U$2.IN@2
- net PC1: no longer P4.@1
- net PC10: no longer P6.@2
- net PC11: no longer P6.@3
- net PC12: no longer P6.@4
- net PC2: no longer P4.@2
- net PC3: no longer P4.@3
- net PC4: no longer P4.@4
- net PC5: no longer P5.@1
- net PC7: no longer P5.@3
- net PC8: no longer P5.@4
- net PC9: no longer P6.@1
- net RF_CE: now also CE.TP, R16.2, U8.PC6; no longer P3.@4, U8.PC0
- net RF_IRQ: now also IRQ.TP; no longer P2.@3
- net RF_MISO: now also MISO.TP; no longer P3.@2
- net RF_MOSI: now also MOSI.TP; no longer P3.@3
- net RF_SCK: now also SCK.TP; no longer P3.@1
- net RF_SS: now also SS.TP; no longer P2.@4
- net SENSOR_SCL: now also R13.1; no longer P2.@1
- net SENSOR_SCL_LV: now also U9.SCL/SCLK; no longer U6.SCL/SCLK
- net SENSOR_SDA: now also R17.1; no longer P2.@2
- net SENSOR_SDA_LV: now also U9.SDA/SDI; no longer U6.SDA/SDI
- net USB_VCC: now also J2.VBUS; no longer J1.A_VBUS, J1.B_VBUS
Other:
- note added: "Input Voltage Source Selector"
- note added: "PA/LNA"
- note added: "Power LED"
- note removed: "BOOT0 should either be pulled up or pulled down NEVER Both Only populate one of these resistors"
